File: arduino-clone.kicad_pcb (KiCad board)
At the start: 4 copper layers, 42.2 x 27.7 mm, 17 parts, among them J1 Serial, J2 Digital Pins, J3 ICSP, J4 I2C, U1 24LC1025, U2 24LC1025, U3 DS13375+, U4 ATMEGA328P-AU, Y1 Crystal 32MHz, Y2 Crystal 16MHz

Commit message: [pcbnew] add silk, add render
Routing:
- added copper zone on In2.Cu, net GNDPWR
Changed lines of the file:
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@@
   (segment (start 142.1567 128.3681) (end 142.1567 128.143) (width 0.25) (layer F.Cu) (net 24))
   (segment (start 143.357 128.143) (end 142.1567 128.143) (width 0.25) (layer F.Cu) (net 24))
+  (zone (net 2) (net_name GNDPWR) (layer In2.Cu) (hatch edge 0.508)
+    (connect_pads (clearance 0.508))
+    (min_thickness 0.254)
+    (fill yes (arc_segments 32) (thermal_gap 0.508) (thermal_bridge_width 0.508))
+    (polygon
+      (pts
+        (xy 144.653 137.414) (xy 143.764 138.557) (xy 103.378 138.557) (xy 103.251 138.303) (xy 103.251 111.506)
+        (xy 144.653 111.506)
+      )
+    )
+  )
 )
